File: can-pico-2209/can-pico-2209.kicad_pcb (KiCad board)
At the start: 2 copper layers, 82 x 68 mm, 17 parts, among them J1 MERG 12v CBUS, J2 Adafruit CAN Pal, J3 DEBUG, J4 UART0, J5 Pico LHS, J6 Pico RHS, SW1 RESET, U1 LM7805_TO220

Commit message: now has 2209 module wired in
Parts:
- removed J2: Adafruit CAN Pal, Connector_PinHeader_2.54mm:PinHeader_1x07_P2.54mm_Vertical
- removed REF** (x4): MountingHole_3.2mm_M3_Pad, MountingHole:MountingHole_3.2mm_M3_Pad
- added H1: MountingHole, MountingHole:MountingHole_3.2mm_M3, F.Cu at (139.5, 39.0)
- added H2: MountingHole, MountingHole:MountingHole_3.2mm_M3, F.Cu at (231.5, 39.0)
- added H3: MountingHole, MountingHole:MountingHole_3.2mm_M3, F.Cu at (231.5, 99.0)
- added H4: MountingHole, MountingHole:MountingHole_3.2mm_M3, F.Cu at (139.5, 99.0)
- added R1: 1K, Resistor_THT:R_Axial_DIN0207_L6.3mm_D2.5mm_P10.16mm_Horizontal, F.Cu at (198.0, 75.0)
- added U2: Can-Pal, Adafruit:CAN-Pal, F.Cu at (186.2, 49.7)
- added U3: ~, Adafruit:Adafruit 2209, F.Cu at (197.1, 91.1)
- moved C1 14.1 mm to (220.1, 78.5)
- moved C2 14.1 mm to (220.1, 88.0)
- moved D1 14.1 mm to (227.1, 73.5)
- moved D2 14.1 mm to (227.1, 46.4)
- moved U1 14.1 mm to (227.1, 80.5)
Routing:
- net Net-(A1-GPIO9): track 5.55 -> 94.5 mm
- net Net-(A1-GPIO8): track 5.55 -> 92.1 mm, vias 0 -> 1
- net Net-(A1-GPIO5): track 5.55 -> 76.8 mm
- net Net-(A1-GPIO6): track 5.55 -> 69.4 mm
- net Net-(A1-GPIO15): track 5.55 -> 68.7 mm
- net Net-(A1-GPIO14): track 5.55 -> 58.3 mm
- net Net-(A1-GPIO7): track 5.55 -> 53.3 mm
- net Net-(A1-GPIO21): track 5.55 -> 41.8 mm
- net Net-(A1-3V3): track 34.1 -> 65.8 mm
- net GND: track 47.5 -> 73.4 mm
- net Net-(A1-VSYS): track 45.2 -> 58.6 mm
- net Net-(A1-GPIO20): track 5.55 -> 16.5 mm
- net Net-(J1-CANH): track 13.7 -> 20.6 mm
- net Net-(D1-A): track 27.9 -> 34.7 mm
- net Net-(J1-CANL): track 20.7 -> 15.5 mm
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Other:
- board size 82 x 68 mm -> 100 x 68 mm
- board text added: "John McAleely Can Pico 2209"
- board text removed: "John McAleely 12v Pico + CAN"
